File: Prototypes/PWM Ramp Gen Prototype/rampgen_sqin.kicad_sch (KiCad schematic)
At the start: 19 parts, among them U1 HFBR-2521Z, U2 AFBR-1528CZ

Commit message: Finishing layout
Connections:
- net at U1.5 (MNT): no longer U1.6 (MNT)
- net at U2.5 (MNT): no longer U2.6 (MNT)
- no-connect marks 2 -> 4
Changed lines of the file:
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@@
   (junction (at 149.86 140.97) (diameter 0) (color 0 0 0 0)
   )
+  (no_connect (at 85.09 92.71))
+  (no_connect (at 85.09 153.67))
   (no_connect (at 85.09 95.25))
   (no_connect (at 85.09 156.21))
