File: Prototypes/PWM Ramp Gen Prototype/rampgen_servo_amp.kicad_sch (KiCad schematic)
At the start: 10 parts

Commit message: Comparator and Op-amp tweaks for BOM consolidation; final layout
Parts:
- removed TP? (x3): -, TestPoint:TestPoint_Pad_D2.0mm, symbol Custom-LogicIC:TestPoint
- removed U?: AD8602, Package_SO:MSOP-8_3x3mm_P0.65mm, symbol Custom-AnalogIC:AD8602
- added U10: AD8601, Package_TO_SOT_SMD:SOT-23-6_Handsoldering, symbol Custom-AnalogIC:AD8601
- renumbered C14 to C16, R17 to R19, R18 to R20, R19 to R21, R20 to R22
Connections:
- net V_{SERVO}: now also U10.1
- net at C?.1, R21.2, R22.1: now also U10.4 (-)
- net at C16.1, R19.2, R20.1: now also U10.3 (+)
